Commit message: Add files via upload

File: urdf/atlas_v5.urdf (robot description, URDF)
Before this commit: robot drc_skeleton, 44 links, 43 joints
Joints:
- removed joint pZtp
- removed joint pxtpy
- removed joint pytpz
- removed joint rxtry
- removed joint rytrz
- removed joint rztpx
- removed joint wtrx
- added joint con_to_pel: type fixed, parent rot_z, child pelvis, origin xyz=0 0 0 rpy=0 0 0, axis 0 0 0
- added joint mov_x: type prismatic, parent world, child pris_x, origin xyz=0 0 0 rpy=0 0 0, axis 1 0 0, limit lower=0 upper=2.35637 effort=890 velocity=12
- added joint mov_y: type prismatic, parent pris_x, child pris_y, origin xyz=0 0 0 rpy=0 0 0, axis 0 1 0, limit lower=0 upper=2.35637 effort=890 velocity=12
- added joint mov_z: type prismatic, parent pris_y, child pris_z, origin xyz=0 0 0 rpy=0 0 0, axis 0 0 1, limit lower=0 upper=2.35637 effort=890 velocity=12
- added joint rotate_x: type continuous, parent pris_z, child rot_x, origin xyz=0 0 0 rpy=0 0 0, axis 1 0 0, limit lower=0 upper=2.35637 effort=890 velocity=12
- added joint rotate_y: type continuous, parent rot_x, child rot_y, origin xyz=0 0 0 rpy=0 0 0, axis 0 1 0, limit lower=0 upper=2.35637 effort=890 velocity=12
- added joint rotate_z: type continuous, parent rot_y, child rot_z, origin xyz=0 0 0 rpy=0 0 0, axis 0 0 1, limit lower=0 upper=2.35637 effort=890 velocity=12

Commit message: no changes

File: urdf/atlas_v5.urdf (robot description, URDF)
Before this commit: robot drc_skeleton, 44 links, 43 joints
Links:
- link world: mass 3.751 -> None

Commit message: chest is now the tip position!

File: urdf/atlas_v5.urdf (robot description, URDF)
Before this commit: robot drc_skeleton, 44 links, 43 joints
Links:
- added link chest, mass 3.751
Joints:
- added joint chest_creator: type fixed, parent utorso, child chest, origin xyz=0 0 0.57 rpy=0 0 0, axis 0 0 0, limit lower=-2 upper=2 effort=275 velocity=12

Commit message: Pushup without weighted tasks, but with center as chest

File: urdf/atlas_v5.urdf (robot description, URDF)
Before this commit: robot drc_skeleton, 45 links, 44 joints
Joints:
- joint chest_creator: origin xyz=0 0 0.57 rpy=0 0 0 -> xyz=0 0 0.37 rpy=0 0 0
